File: PCB/ESP32DEV.kicad_pcb (KiCad board)
At the start: 2 copper layers, 34.7 x 43.8 mm, 32 parts, among them J1 USB_C_Receptacle_USB2.0_16P, J2 Conn_01x18_Pin, J3 Conn_01x18_Pin, J5 Conn_01x04_Pin, J6 Conn_01x02_Pin, Q1 AO3401A, SW1 SW_Push, SW2 SW_Push, U2 AP63203WU, U5 ESP32-S3-WROOM-1

Commit message: Add files via upload
Other:
- board text added: "ESP32 DEVBOARD"
Changed lines of the file:
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@@
+		)
+	)
+	(gr_text "ESP32 DEVBOARD"
+		(at 139.3 87.24 0)
+		(layer "B.SilkS")
+		(effects
+			(font
+				(size 2 2)
+				(thickness 0.5)
+				(bold yes)
+			)
+			(justify left bottom mirror)
 		)
 	)

Commit message: Add files via upload
Parts:
- removed C1: 2u2, Capacitor_SMD:C_0201_0603Metric
- removed R5: 100R, Resistor_SMD:R_0603_1608Metric
- added D4: 1N4001, Diode_THT:D_DO-41_SOD81_P2.54mm_Vertical_AnodeUp, F.Cu at (122.4, 112.7)
- added L1: 4.7uh, Inductor_SMD:L_0603_1608Metric, F.Cu at (127.3, 109.5)
- added L2: 2.2uh, Inductor_SMD:L_0603_1608Metric, F.Cu at (123.9, 110.2)
- C2: value 2u2 -> 47uf
- C3: value 2u2 -> 10uf
- C4: value 100n -> 100nf
- C5: value 22u -> 22uf
- C6: value 100n -> 22uf
- R1, R2, R3, R4: footprint Resistor_SMD:R_0201_0603Metric_Pad0.64x0.40mm_HandSolder -> Resistor_SMD:R_0603_1608Metric
- moved C2 2.39 mm to (124.5, 112.4)
- moved C3 2.30 mm to (125.3, 112.4)
- moved R3 0.89 mm to (117.1, 117.8)
- moved R4 0.76 mm to (121.9, 118.1)
- moved R2 0.47 mm to (120.3, 118.1)
- moved R1 0.42 mm to (118.8, 118.1)
- renumbered C5x to C5(1uf)1, C6x to C6(100nf)1, R1x to R1(10k)1, R2x to R2(100R)1
Connections:
- net I022 renamed I014
- net I024 renamed I047
- net I025 renamed I048
- net I026 renamed I045
- net I033 renamed I040
- net I034 renamed I041
- net Power renamed +5V
- C4 pad 1: 3.3V -> +3.3V
- C5 pad 1: 3.3V -> +3.3V
- C6 pad 1: 3.3V -> +3.3V
- J2 pad 10: I010 -> I017
- J2 pad 11: I011 -> I018
- J2 pad 12: I012 -> I08
- J2 pad 15: I015 -> I03
- J2 pad 16: I016 -> I046
- J2 pad 17: I017 -> I09
- J2 pad 18: I018 -> I010
- J2 pad 2: 3.3V -> +3.3V
- J2 pad 8: I08 -> I015
- J2 pad 9: I09 -> I016
- J3 pad 1: I023 -> I021
- J3 pad 10: I032 -> I039
- J3 pad 13: I035 -> I042
- J3 pad 14: I036 -> TX
- J3 pad 15: I037 -> RX
- J3 pad 16: I038 -> I01
- J3 pad 17: I039 -> I02
- J3 pad 6: I028 -> I035
- J3 pad 7: I029 -> I036
- J3 pad 8: I030 -> I037
- J3 pad 9: I031 -> I038
- J5 pad 2: I021 -> I013
- J5 pad 3: I020 -> I012
- J5 pad 4: I019 -> I011
- R1(10k)1 pad 1: 3.3V -> +3.3V
- R6 pad 1: 3.3V -> +3.3V
- R8 pad 2: I019 -> I011
- U2 pad 1: 3.3V -> Net-(U2-FB)
- U2 pad 5: 3.3V -> +3.3V
- U5 pad 10: I010 -> I017
- U5 pad 11: I011 -> I018
- U5 pad 12: I012 -> I08
- U5 pad 15: I015 -> I03
- U5 pad 16: I016 -> I046
- U5 pad 17: I017 -> I09
- U5 pad 18: I018 -> I010
- U5 pad 19: I019 -> I011
- U5 pad 2: 3.3V -> +3.3V
- U5 pad 20: I020 -> I012
- U5 pad 21: I021 -> I013
- U5 pad 23: I023 -> I021
- U5 pad 28: I028 -> I035
- U5 pad 29: I029 -> I036
- U5 pad 30: I030 -> I037
- U5 pad 31: I031 -> I038
- U5 pad 32: I032 -> I039
- U5 pad 35: I035 -> I042
- U5 pad 36: I037 -> RX
- U5 pad 37: I036 -> TX
- U5 pad 38: I039 -> I02
- U5 pad 39: I038 -> I01
- U5 pad 8: I08 -> I015
- U5 pad 9: I09 -> I016
Routing:
- net 3.3V: track 50.3 -> 0.00 mm, vias 2 -> 0
- net +3.3V: track 0.00 -> 47.6 mm, vias 0 -> 2
- net I019: track 25.1 -> 0.00 mm, vias 1 -> 0
- net I023: track 21.4 -> 0.00 mm, vias 1 -> 0
- net I020: track 17.8 -> 0.00 mm, vias 1 -> 0
- net I046: track 0.00 -> 17.8 mm, vias 0 -> 2
- net I013: track 0.00 -> 17.7 mm, vias 0 -> 1
- net I03: track 0.00 -> 15.9 mm, vias 0 -> 2
- net I011: track 10.9 -> 25.1 mm, vias 0 -> 1
- net _D-: track 26.4 -> 38.7 mm, vias 0 -> 2
- net I028: track 12.0 -> 0.00 mm
- net I010: track 9.84 -> 21.6 mm, vias 0 -> 2
- net I029: track 11.1 -> 0.00 mm
- net I018: track 21.6 -> 10.9 mm, vias 2 -> 0
- net I030: track 10.4 -> 0.00 mm
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Other:
- board text added: "IO1"
- board text added: "IO10"
- board text added: "IO11"
- board text added: "IO12"
- board text added: "IO2"
- board text added: "IO3"
- board text added: "IO40"
- board text added: "IO41"
- board text added: "IO42"
- board text added: "IO45"
- board text added: "IO46"
- board text added: "IO47"
- board text added: "IO48"
- board text added: "IOTX"
- board text added: "RX"
- board text removed: "IO19"
- board text removed: "IO20"
- board text removed: "IO22"
- board text removed: "IO23"
- board text removed: "IO24"
- board text removed: "IO25"
- board text removed: "IO26"
- board text removed: "IO28"
- board text removed: "IO29"
- board text removed: "IO30"
- board text removed: "IO31"
- board text removed: "IO32"
- board text removed: "IO33"
- board text removed: "IO34"

Commit message: Add files via upload
Parts:
- renumbered C5(1uf)1 to C5Z, C6(100nf)1 to C6Z, R1(10k)1 to R1Z, R2(100R)1 to R2Z
Other:
- outline, holes or cut-outs redrawn
Changed lines of the file:
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@@
 		(descr "Capacitor SMD 0805 (2012 Metric), square (rectangular) end terminal, IPC-7351 nominal, (Body size source: IPC-SM-782 page 76, https://www.pcb-3d.com/wordpress/wp-content/uploads/ipc-sm-782a_amendment_1_and_2.pdf, https://docs.google.com/spreadsheets/d/1BsfQQcO9C6DZCsRaXUlFlo91Tg2WpOkGARC1WS5S8t0/edit?usp=sharing), generated with kicad-footprint-generator")
 		(tags "capacitor")
-		(property "Reference" "C6(100nf)1"
-			(at -2.11 0.25 180)
+		(property "Reference" "C6Z"
+			(at -2.735 0.45 180)
 			(layer "F.SilkS")
 			(effects
@@
 		(descr "Resistor SMD 0805 (2012 Metric), square (rectangular) end terminal, IPC-7351 nominal, (Body size source: IPC-SM-782 page 72, https://www.pcb-3d.com/wordpress/wp-content/uploads/ipc-sm-782a_amendment_1_and_2.pdf), generated with kicad-footprint-generator")
 		(tags "resistor")
-		(property "Reference" "R1(10k)1"
-			(at 2.0725 -0.14 180)
+		(property "Reference" "R1Z"
+			(at 2.1875 0.025 180)
 			(layer "F.SilkS")
 			(effects
@@
 		(tags "capacitor")
 		(property "Reference" "C4"
-			(at 1.69 0.06 90)
+			(at 1.6225 -0.1325 90)
 			(layer "F.SilkS")
 			(effects
@@
 		(tags "SPST Button Switch")
 		(property "Reference" "SW1"
-			(at 0 -2.6 0)
+			(at 0.63 -2.225 0)
 			(layer "F.SilkS")
 			(effects
 				(font
-					(size 1 1)
-					(thickness 0.15)
+					(size 0.5 0.5)
+					(thickness 0.125)
 				)
 			)
@@
 		(tags "LED")
 		(property "Reference" "D3"
-			(at -1.435 -0.12 90)
+			(at -1.095 -0.075 90)
 			(layer "F.SilkS")
 			(effects
@@
 		(tags "resistor handsolder")
 		(property "Reference" "R6"
-			(at 1.4475 0.05 90)
+			(at 1.6225 0.1 90)
 			(layer "F.SilkS")
 			(effects
@@
 		(descr "Capacitor SMD 0805 (2012 Metric), square (rectangular) end terminal, IPC-7351 nominal, (Body size source: IPC-SM-782 page 76, https://www.pcb-3d.com/wordpress/wp-content/uploads/ipc-sm-782a_amendment_1_and_2.pdf, https://docs.google.com/spreadsheets/d/1BsfQQcO9C6DZCsRaXUlFlo91Tg2WpOkGARC1WS5S8t0/edit?usp=sharing), generated with kicad-footprint-generator")
 		(tags "capacitor")
-		(property "Reference" "C5(1uf)1"
-			(at -2.14 0.14 180)
+		(property "Reference" "C5Z"
+			(at -2.835 0.085 180)
 			(layer "F.SilkS")
 			(effects
@@
 		(tags "SPST Button Switch")
 		(property "Reference" "SW2"
-			(at -3.55 0.17 180)
+			(at -3.99 0.17 180)
 			(layer "F.SilkS")
 			(effects
@@
 		(descr "Resistor SMD 0805 (2012 Metric), square (rectangular) end terminal, IPC-7351 nominal, (Body size source: IPC-SM-782 page 72, https://www.pcb-3d.com/wordpress/wp-content/uploads/ipc-sm-782a_amendment_1_and_2.pdf), generated with kicad-footprint-generator")
 		(tags "resistor")
-		(property "Reference" "R2(100R)1"
+		(property "Reference" "R2Z"
 			(at -0.1 1.29 0)
 			(layer "F.SilkS")
@@
 		)
 	)
-	(gr_rect
-		(start 109.23 83.28)
-		(end 143.97 127.05)
+	(gr_line
+		(start 109.23 126.05)
+		(end 109.23 84.28)
+		(stroke
+			(width 0.05)
+			(type default)
+		)
+		(layer "Edge.Cuts")
+	)
+	(gr_line
+		(start 143.97 84.28)
+		(end 143.97 126.05)
+		(stroke
+			(width 0.05)
+			(type default)
+		)
+		(layer "Edge.Cuts")
+	)
+	(gr_line
+		(start 110.23 83.28)
+		(end 142.97 83.28)
+		(stroke
+			(width 0.05)
+			(type default)
+		)
+		(layer "Edge.Cuts")
+	)
+	(gr_arc
+		(start 142.97 83.28)
+		(mid 143.677107 83.572893)
+		(end 143.97 84.28)
+		(stroke
+			(width 0.05)
+			(type default)
+		)
+		(layer "Edge.Cuts")
+	)
+	(gr_arc
+		(start 143.97 126.05)
+		(mid 143.677107 126.757107)
+		(end 142.97 127.05)
+		(stroke
+			(width 0.05)
+			(type default)
+		)
+		(layer "Edge.Cuts")
+	)
+	(gr_line
+		(start 142.97 127.05)
+		(end 110.23 127.05)
+		(stroke
+			(width 0.05)
+			(type default)
+		)
+		(layer "Edge.Cuts")
+	)
+	(gr_arc
+		(start 110.23 127.05)
+		(mid 109.522893 126.757107)
+		(end 109.23 126.05)
+		(stroke
+			(width 0.05)
+			(type solid)
+		)
+		(layer "Edge.Cuts")
+	)
+	(gr_arc
+		(start 109.23 84.28)
+		(mid 109.522893 83.572893)
+		(end 110.23 83.28)
 		(stroke
 			(width 0.05)
 			(type default)
 		)
-		(fill no)
 		(layer "Edge.Cuts")
 	)
